Commit message: fisheye

File: urdf/c5.xacro (robot description, xacro)
@@ -23,4 +23,5 @@
   <xacro:property name="mesh_file" value="package://aeroscan_uav_simulation/meshes/untitled.dae" />
   <xacro:property name="mass" value="5.266" />
+  <xacro:property name="mass_arm" value="0.01" /> <!-- [kg] -->
   <!-- <xacro:property name="mass" value="1.5" /> -->
   <xacro:property name="body_width" value="1.5" />

File: urdf/component_snippets.xacro (robot description, xacro)
@@ -29,4 +29,94 @@
 	<waitToRecordBag>${wait_to_record_bag}</waitToRecordBag>
       </plugin>
+    </gazebo>
+  </xacro:macro>
+  <!-- Macro to add a camera. -->
+  <xacro:macro name="camera_fisheye"
+    params="namespace parent_link camera_suffix frame_rate
+      horizontal_fov image_width image_height min_distance
+      max_distance noise_mean noise_stddev enable_visual *geometry *origin">
+    <link name="${namespace}/camera_${camera_suffix}_link">
+      <collision>
+        <origin xyz="0 0 0" rpy="0 0 0" />
+        <geometry>
+          <xacro:insert_block name="geometry" />
+        </geometry>
+      </collision>
+      <xacro:if value="${enable_visual}">
+        <visual>
+          <origin xyz="0 0 0" rpy="0 ${pi/2} 0" />
+          <geometry>
+            <xacro:insert_block name="geometry" />
+          </geometry>
+          <material name="red" />
+        </visual>
+      </xacro:if>
+      <inertial>
+        <mass value="1e-5" />
+        <origin xyz="0 0 0" rpy="0 0 0" />
+        <inertia ixx="1e-6" ixy="0" ixz="0" iyy="1e-6" iyz="0" izz="1e-6" />
+      </inertial>
+    </link>
+    <joint name="${namespace}/camera_${camera_suffix}_joint" type="fixed">
+      <xacro:insert_block name="origin" />
+      <parent link="${parent_link}" />
+      <child link="${namespace}/camera_${camera_suffix}_link" />
+    </joint>
+    <link name="${namespace}/camera_${camera_suffix}_optical_link" />
+    <joint name="${namespace}/camera_${camera_suffix}_optical_joint" type="fixed" >
+      <origin xyz="0 0 0" rpy="${-pi/2} 0 ${-pi/2}" />
+      <parent link="${namespace}/camera_${camera_suffix}_link" />
+      <child link="${namespace}/camera_${camera_suffix}_optical_link" />
+    </joint>
+    <gazebo reference="${namespace}/camera_${camera_suffix}_link">
+      <sensor type="wideanglecamera" name="${namespace}_camera_${camera_suffix}">
+        <update_rate>${frame_rate}</update_rate>
+        <camera name="head">
+          <horizontal_fov>${horizontal_fov}</horizontal_fov>
+          <image>
+            <width>${image_width}</width>
+            <height>${image_height}</height>
+          </image>
+          <clip>
+            <near>${min_distance}</near>
+            <far>${max_distance}</far>
+          </clip>
+          <!-- A new section named `lens`. -->
+           <lens>
+             <!-- type element is mandatory -->
+             <type>custom</type>
+             <!-- manually defined mapping function r = c1*f*fun(theta/c2 + c3) -->
+             <!-- More information here: https://en.wikipedia.org/wiki/Fisheye_lens#Mapping_function -->
+             <custom_function>
+               <c1>1.05</c1>   <!-- linear scaling -->
+               <c2>4</c2>      <!-- angle scaling -->
+               <f>1.0</f>      <!-- one more scaling parameter -->
+               <fun>tan</fun>  <!-- one of sin,tan,id -->
+             </custom_function>
+             <!-- if it is set to `true` your horizontal FOV will ramain as defined -->
+             <!-- othervise it depends on lens type and custom function, if there is one -->
+             <scale_to_hfov>true</scale_to_hfov>
+             <!-- clip everything that is outside of this angle -->
+             <cutoff_angle>3.1415</cutoff_angle>
+             <!-- resolution of the cubemap texture, the highter it is - the sharper is your image -->
+             <env_texture_size>512</env_texture_size>
+           </lens>
+        </camera>
+        <plugin name="${namespace}_camera_${camera_suffix}_controller" filename="libgazebo_ros_camera.so">
+          <robotNamespace>${namespace}</robotNamespace>
+          <alwaysOn>true</alwaysOn>
+          <updateRate>${frame_rate}</updateRate>
+          <cameraName>camera_${camera_suffix}</cameraName>
+          <imageTopicName>image_raw</imageTopicName>
+          <cameraInfoTopicName>camera_info</cameraInfoTopicName>
+          <frameName>camera_${camera_suffix}_link</frameName>
+          <hackBaseline>0.0</hackBaseline>
+          <distortionK1>0.0</distortionK1>
+          <distortionK2>0.0</distortionK2>
+          <distortionK3>0.0</distortionK3>
+          <distortionT1>0.0</distortionT1>
+          <distortionT2>0.0</distortionT2>
+        </plugin>
+      </sensor>
     </gazebo>
   </xacro:macro>

File: urdf/firefly.xacro (robot description, xacro)
@@ -21,4 +21,5 @@
   <xacro:property name="rotor_velocity_slowdown_sim" value="10" />
   <xacro:property name="use_mesh_file" value="true" />
+  <xacro:property name="mass_arm" value="0.01" /> <!-- [kg] -->
   <xacro:property name="mesh_file" value="package://aeroscan_uav_simulation/meshes/firefly.dae" />
   <xacro:property name="mass" value="1.5" /> <!-- [kg] -->

Commit message: stitching and mesh disable

File: urdf/c5.xacro (robot description, xacro)
@@ -415,5 +415,6 @@
           <origin xyz="-0.0 0 0" rpy="1.57 0 3.1415"/>
           <geometry>
-              <mesh filename="file:///$(find aeroscan_uav_simulation)/meshes/scanstation_c5.dae" scale="0.001 0.001 0.001"/>
+              <!-- <mesh filename="file:///$(find aeroscan_uav_simulation)/meshes/scanstation_c5.dae" scale="0.001 0.001 0.001"/> -->
+              <cylinder length="0.0001" radius="0.0001"/>
           </geometry>
       </visual>
@@ -421,5 +422,6 @@
           <origin xyz="-0.0 -0. 0" rpy="1.57 0 3.1415"/>
           <geometry>
-              <mesh filename="file:///$(find aeroscan_uav_simulation)/meshes/scanstation_c5.stl" scale="0.001 0.001 0.001"/>
+              <!-- <mesh filename="file:///$(find aeroscan_uav_simulation)/meshes/scanstation_c5.stl" scale="0.001 0.001 0.001"/> -->
+              <cylinder length="0.0001" radius="0.0001"/>
           </geometry>
       </collision>
@@ -448,11 +450,14 @@
                       <samples>512</samples>
                       <resolution>1</resolution>
-                      <min_angle>-0.78539816339</min_angle> <!-- Be sure the angle between min and max angle is > 1.5708 -->
+                      <min_angle>-0.78539816339</min_angle>
                       <max_angle>0.78539816339</max_angle>
+                      <!-- <min_angle>-3.14159265359</min_angle>
+                      <max_angle>3.14159265359</max_angle> -->
                   </horizontal>
               </scan>
               <range>
-                  <min>0.15</min>
-                  <max>130.0</max>
+                  <!-- <min>0.15</min> -->
+                  <min>0.5</min>
+                  <max>250.0</max>
                   <resolution>0.01</resolution>
               </range>

File: urdf/multirotor_base_firefly.xacro (robot description, xacro)
@@ -53,5 +53,5 @@
           </xacro:if>
           <xacro:unless value="${use_mesh_file}">
-            <box size="${body_width} ${body_width} ${body_height}"/>
+            <cylinder length="0.0001" radius="0.0001"/>
           </xacro:unless>
         </geometry>
@@ -60,5 +60,6 @@
         <origin xyz="0 0 0.35" rpy="0 0 0" />
         <geometry>
-          <box size="${body_width} ${body_width} 0.1" /> <!-- [m] [m] [m] -->
+          <!-- <box size="${body_width} ${body_width} 0.1" />  -->
+          <cylinder length="0.0001" radius="0.0001"/>
         </geometry>
       </collision>
@@ -100,5 +101,4 @@
       <visual>
         <geometry>
-          <!-- <cylinder length="0.005" radius="${radius_rotor}"/> --> <!-- [m] -->
           <xacro:if value="${use_own_mesh}">
             <mesh filename="${mesh}"
@@ -106,7 +106,5 @@
           </xacro:if>
           <xacro:unless value="${use_own_mesh}">
-            <mesh filename="package://rotors_description/meshes/propeller_${direction}.dae"
-              scale="${radius_rotor} ${radius_rotor} ${radius_rotor}" /> <!-- The propeller meshes have a radius of 1m -->
-            <!-- <box size="${2*radius_rotor} 0.01 0.005"/> -->
+            <cylinder length="0.0001" radius="0.0001"/>
           </xacro:unless>
         </geometry>

Commit message: adjustments

File: urdf/c5.xacro (robot description, xacro)
@@ -31,7 +31,4 @@
   <xacro:property name="rotor_offset_top" value="0.4" />
   <xacro:property name="radius_rotor" value="0.25" />
-  <!-- <xacro:property name="mass_rotor" value="0.05" /> -->
-  <!-- <xacro:property name="radius_rotor" value="0.1" /> -->
-  <!-- <xacro:property name="rotor_offset_top" value="0.023" />  -->
   <xacro:property name="arm_length_front_x" value="0.745" /> <!-- [m] -->
   <xacro:property name="arm_length_back_x" value="0.745" /> <!-- [m] -->
@@ -49,8 +46,4 @@
   <xacro:property name="rotor_drag_coefficient" value="8.06428e-05" />
   <xacro:property name="rolling_moment_coefficient" value="0.000001" />
-  <!-- Property Blocks -->
-  <!-- <xacro:property name="body_inertia">
-    <inertia ixx="88.12874706" ixy="3.049735432" ixz="-0.002397487" iyy="2.933980791" iyz="3.332416221" izz="88.102728321" />
-  </xacro:property> -->
   <xacro:property name="body_inertia">
     <inertia ixx="0.0347563" ixy="0.0" ixz="0.0" iyy="0.0458929" iyz="0.0" izz="0.0977" /> <!-- [kg.m^2] [kg.m^2] [kg.m^2] [kg.m^2] [kg.m^2] [kg.m^2] -->
@@ -61,5 +54,5 @@
   </xacro:property>
   <!-- Included URDF Files -->
-  <xacro:include filename="$(find aeroscan_uav_simulation)/urdf/multirotor_base_firefly.xacro" />
+  <xacro:include filename="$(find aeroscan_uav_simulation)/urdf/multirotor_base.xacro" />
   <!-- Instantiate multirotor_base_macro once -->
   <xacro:multirotor_base_macro
@@ -73,172 +66,4 @@
     <xacro:insert_block name="body_inertia" />
   </xacro:multirotor_base_macro>
-  <!-- <xacro:vertical_rotor
-    robot_namespace="${namespace}"
-    suffix="front_left"
-    direction="ccw"
-    motor_constant="${motor_constant}"
-    moment_constant="${moment_constant}"
-    parent="${namespace}/base_link"
-    mass_rotor="${mass_rotor}"
-    radius_rotor="${radius_rotor}"
-    time_constant_up="${time_constant_up}"
-    time_constant_down="${time_constant_down}"
-    max_rot_velocity="${max_rot_velocity}"
-    motor_number="0"
-    rotor_drag_coefficient="${rotor_drag_coefficient}"
-    rolling_moment_coefficient="${rolling_moment_coefficient}"
-    color="Blue"
-    use_own_mesh="false"
-    mesh="">
-    <origin xyz="${arm_length*0.3826834323650898} ${arm_length*0.9238795325112867} ${rotor_offset_top}" rpy="0 0 0" />
-    <xacro:insert_block name="rotor_inertia" />
-  </xacro:vertical_rotor>
-  <xacro:vertical_rotor
-    robot_namespace="${namespace}"
-    suffix="front_left"
-    direction="cw"
-    motor_constant="${motor_constant}"
-    moment_constant="${moment_constant}"
-    parent="${namespace}/base_link"
-    mass_rotor="${mass_rotor}"
-    radius_rotor="${radius_rotor}"
-    time_constant_up="${time_constant_up}"
-    time_constant_down="${time_constant_down}"
-    max_rot_velocity="${max_rot_velocity}"
-    motor_number="1"
-    rotor_drag_coefficient="${rotor_drag_coefficient}"
-    rolling_moment_coefficient="${rolling_moment_coefficient}"
-    color="Red"
-    use_own_mesh="false"
-    mesh="">
-    <origin xyz="${arm_length*0.9238795325112867} ${arm_length*0.3826834323650898} ${rotor_offset_top}" rpy="0 0 0" />
-    <xacro:insert_block name="rotor_inertia" />
-  </xacro:vertical_rotor>
-  <xacro:vertical_rotor
-    robot_namespace="${namespace}"
-    suffix="left"
-    direction="ccw"
-    motor_constant="${motor_constant}"
-    moment_constant="${moment_constant}"
-    parent="${namespace}/base_link"
-    mass_rotor="${mass_rotor}"
-    radius_rotor="${radius_rotor}"
-    time_constant_up="${time_constant_up}"
-    time_constant_down="${time_constant_down}"
-    max_rot_velocity="${max_rot_velocity}"
-    motor_number="2"
-    rotor_drag_coefficient="${rotor_drag_coefficient}"
-    rolling_moment_coefficient="${rolling_moment_coefficient}"
-    color="Blue"
-    use_own_mesh="false"
-    mesh="">
-    <origin xyz="${arm_length*0.9238795325112867} -${arm_length*0.3826834323650898} ${rotor_offset_top}" rpy="0 0 0" />
-    <xacro:insert_block name="rotor_inertia" />
-  </xacro:vertical_rotor>
-  <xacro:vertical_rotor
-    robot_namespace="${namespace}"
-    suffix="front_left"
-    direction="cw"
-    motor_constant="${motor_constant}"
-    moment_constant="${moment_constant}"
-    parent="${namespace}/base_link"
-    mass_rotor="${mass_rotor}"
-    radius_rotor="${radius_rotor}"
-    time_constant_up="${time_constant_up}"
-    time_constant_down="${time_constant_down}"
-    max_rot_velocity="${max_rot_velocity}"
-    motor_number="3"
-    rotor_drag_coefficient="${rotor_drag_coefficient}"
-    rolling_moment_coefficient="${rolling_moment_coefficient}"
-    color="Red"
-    use_own_mesh="false"
-    mesh="">
-    <origin xyz="${arm_length*0.3826834323650898} -${arm_length*0.9238795325112867} ${rotor_offset_top}" rpy="0 0 0" />
-    <xacro:insert_block name="rotor_inertia" />
-  </xacro:vertical_rotor>
-  <xacro:vertical_rotor
-    robot_namespace="${namespace}"
-    suffix="left"
-    direction="ccw"
-    motor_constant="${motor_constant}"
-    moment_constant="${moment_constant}"
-    parent="${namespace}/base_link"
-    mass_rotor="${mass_rotor}"
-    radius_rotor="${radius_rotor}"
-    time_constant_up="${time_constant_up}"
-    time_constant_down="${time_constant_down}"
-    max_rot_velocity="${max_rot_velocity}"
-    motor_number="4"
-    rotor_drag_coefficient="${rotor_drag_coefficient}"
-    rolling_moment_coefficient="${rolling_moment_coefficient}"
-    color="Blue"
-    use_own_mesh="false"
-    mesh="">
-    <origin xyz="-${arm_length*0.3826834323650898} -${arm_length*0.9238795325112867} ${rotor_offset_top}" rpy="0 0 0" />
-    <xacro:insert_block name="rotor_inertia" />
-  </xacro:vertical_rotor>
-  <xacro:vertical_rotor
-    robot_namespace="${namespace}"
-    suffix="front_left"
-    direction="cw"
-    motor_constant="${motor_constant}"
-    moment_constant="${moment_constant}"
-    parent="${namespace}/base_link"
-    mass_rotor="${mass_rotor}"
-    radius_rotor="${radius_rotor}"
-    time_constant_up="${time_constant_up}"
-    time_constant_down="${time_constant_down}"
-    max_rot_velocity="${max_rot_velocity}"
-    motor_number="5"
-    rotor_drag_coefficient="${rotor_drag_coefficient}"
-    rolling_moment_coefficient="${rolling_moment_coefficient}"
-    color="Red"
-    use_own_mesh="false"
-    mesh="">
-    <origin xyz="-${arm_length*0.9238795325112867} -${arm_length*0.3826834323650898} ${rotor_offset_top}" rpy="0 0 0" />
-    <xacro:insert_block name="rotor_inertia" />
-  </xacro:vertical_rotor>
-  <xacro:vertical_rotor
-    robot_namespace="${namespace}"
-    suffix="left"
-    direction="ccw"
-    motor_constant="${motor_constant}"
-    moment_constant="${moment_constant}"
-    parent="${namespace}/base_link"
-    mass_rotor="${mass_rotor}"
-    radius_rotor="${radius_rotor}"
-    time_constant_up="${time_constant_up}"
-    time_constant_down="${time_constant_down}"
-    max_rot_velocity="${max_rot_velocity}"
-    motor_number="6"
-    rotor_drag_coefficient="${rotor_drag_coefficient}"
-    rolling_moment_coefficient="${rolling_moment_coefficient}"
-    color="Blue"
-    use_own_mesh="false"
-    mesh="">
-    <origin xyz="-${arm_length*0.9238795325112867} ${arm_length*0.3826834323650898} ${rotor_offset_top}" rpy="0 0 0" />
-    <xacro:insert_block name="rotor_inertia" />
-  </xacro:vertical_rotor>
-  <xacro:vertical_rotor
-    robot_namespace="${namespace}"
-    suffix="front_left"
-    direction="cw"
-    motor_constant="${motor_constant}"
-    moment_constant="${moment_constant}"
-    parent="${namespace}/base_link"
-    mass_rotor="${mass_rotor}"
-    radius_rotor="${radius_rotor}"
-    time_constant_up="${time_constant_up}"
-    time_constant_down="${time_constant_down}"
-    max_rot_velocity="${max_rot_velocity}"
-    motor_number="7"
-    rotor_drag_coefficient="${rotor_drag_coefficient}"
-    rolling_moment_coefficient="${rolling_moment_coefficient}"
-    color="Red"
-    use_own_mesh="false"
-    mesh="">
-    <origin xyz="-${arm_length*0.3826834323650898} ${arm_length*0.9238795325112867} ${rotor_offset_top}" rpy="0 0 0" />
-    <xacro:insert_block name="rotor_inertia" />
-  </xacro:vertical_rotor> -->
   <xacro:vertical_rotor
     robot_namespace="${namespace}"
@@ -408,10 +233,10 @@
   <link name="${namespace}/base_link/sensor_link">
       <inertial>
-          <origin xyz="-0.0 -0. 0" rpy="1.57 0 3.1415"/>
+          <origin xyz="0 0 0" rpy="1.57079632679 0 3.14159265359"/>
           <mass value="0.05" />
           <inertia ixx="0.0" ixy="0.0" ixz="0.0" iyy="0.0" iyz="0.0" izz="0.0" />
       </inertial>
       <visual>
-          <origin xyz="-0.0 0 0" rpy="1.57 0 3.1415"/>
+          <origin xyz="0 0 0" rpy="1.57079632679 0 3.14159265359"/>
           <geometry>
               <!-- <mesh filename="file:///$(find aeroscan_uav_simulation)/meshes/scanstation_c5.dae" scale="0.001 0.001 0.001"/> -->
@@ -420,5 +245,5 @@
       </visual>
       <collision>
-          <origin xyz="-0.0 -0. 0" rpy="1.57 0 3.1415"/>
+          <origin xyz="0 0 0" rpy="1.57079632679 0 3.14159265359"/>
           <geometry>
               <!-- <mesh filename="file:///$(find aeroscan_uav_simulation)/meshes/scanstation_c5.stl" scale="0.001 0.001 0.001"/> -->
@@ -430,5 +255,5 @@
   <!-- <xacro:include filename="$(find aeroscan_uav_simulation)/urdf/sensor.urdf.xacro" /> -->
   <joint name="sensor_joint" type="fixed">
-      <origin xyz="0 0 -0.073" rpy="1.57 0 0"/>
+      <origin xyz="0 0 0" rpy="1.57079632679 0 0"/>
       <parent link="${namespace}/base_link"/>
       <child link="${namespace}/base_link/sensor_link"/>
@@ -442,5 +267,5 @@
       <static>true</static>
       <sensor type="gpu_ray" name="leica_sensor">
-          <pose>0.05 0 -0.25 1.57 0 0</pose>
+          <pose>0.0 0 0.0 1.57079632679 0 0</pose>
           <visualize>true</visualize>
           <update_rate>40</update_rate>

File: urdf/multirotor_base.xacro (robot description, xacro)
@@ -47,5 +47,5 @@
       </inertial>
       <visual>
-        <origin xyz="0 0 0" rpy="0 0 0" />
+        <origin xyz="-0.77 -0.82 -0.4" rpy="1.57075 0 1.57075" />
         <geometry>
           <xacro:if value="${use_mesh_file}">
@@ -53,12 +53,19 @@
           </xacro:if>
           <xacro:unless value="${use_mesh_file}">
-            <box size="${body_width} ${body_width} ${body_height}"/> <!-- [m] [m] [m] -->
+            <cylinder length="0.0001" radius="0.0001"/>
           </xacro:unless>
         </geometry>
       </visual>
       <collision>
+        <origin xyz="0 0 0.35" rpy="0 0 0" />
+        <geometry>
+          <!-- <box size="${body_width} ${body_width} 0.1" />  -->
+          <cylinder length="0.0001" radius="0.0001"/>
+        </geometry>
+      </collision>
+      <collision>
         <origin xyz="0 0 0" rpy="0 0 0" />
         <geometry>
-          <box size="${body_width} ${body_width} ${body_height}" /> <!-- [m] [m] [m] -->
+          <box size="${body_width/2.5} ${body_width/2.5} 0.8" /> <!-- [m] [m] [m] -->
         </geometry>
       </collision>
@@ -71,4 +78,7 @@
         <rotorVelocitySlowdownSim>${rotor_velocity_slowdown_sim}</rotorVelocitySlowdownSim>
       </plugin>
+    </gazebo>
+    <gazebo reference="${robot_namespace}/base_link">
+      <material>Gazebo/Black</material>
     </gazebo>
   </xacro:macro>
@@ -86,18 +96,15 @@
     <link name="${robot_namespace}/rotor_${motor_number}">
       <inertial>
-        <mass value="${mass_rotor}" /> <!-- [kg] -->
+        <mass value="${mass_rotor}" />
         <xacro:insert_block name="inertia" />
       </inertial>
       <visual>
         <geometry>
-          <!-- <cylinder length="0.005" radius="${radius_rotor}"/> --> <!-- [m] -->
           <xacro:if value="${use_own_mesh}">
             <mesh filename="${mesh}"
-              scale="1 1 1" />
+              scale="10 10 10" />
           </xacro:if>
           <xacro:unless value="${use_own_mesh}">
-            <mesh filename="package://rotors_description/meshes/propeller_${direction}.dae"
-              scale="${radius_rotor} ${radius_rotor} ${radius_rotor}" /> <!-- The propeller meshes have a radius of 1m -->
-            <!-- <box size="${2*radius_rotor} 0.01 0.005"/> -->
+            <cylinder length="0.0001" radius="0.0001"/>
           </xacro:unless>
         </geometry>

Commit message: ros noetic

File: urdf/c5.xacro (robot description, xacro)
@@ -240,6 +240,6 @@
           <origin xyz="0 0 0" rpy="1.57079632679 0 3.14159265359"/>
           <geometry>
-              <!-- <mesh filename="file:///$(find aeroscan_uav_simulation)/meshes/scanstation_c5.dae" scale="0.001 0.001 0.001"/> -->
-              <cylinder length="0.0001" radius="0.0001"/>
+              <mesh filename="file:///$(find aeroscan_uav_simulation)/meshes/scanstation_c5.dae" scale="0.001 0.001 0.001"/>
+              <!-- <cylinder length="0.0001" radius="0.0001"/> -->
           </geometry>
       </visual>
@@ -247,6 +247,6 @@
           <origin xyz="0 0 0" rpy="1.57079632679 0 3.14159265359"/>
           <geometry>
-              <!-- <mesh filename="file:///$(find aeroscan_uav_simulation)/meshes/scanstation_c5.stl" scale="0.001 0.001 0.001"/> -->
-              <cylinder length="0.0001" radius="0.0001"/>
+              <mesh filename="file:///$(find aeroscan_uav_simulation)/meshes/scanstation_c5.stl" scale="0.001 0.001 0.001"/>
+              <!-- <cylinder length="0.0001" radius="0.0001"/> -->
           </geometry>
       </collision>

File: urdf/multirotor_base.xacro (robot description, xacro)
@@ -102,9 +102,11 @@
         <geometry>
           <xacro:if value="${use_own_mesh}">
-            <mesh filename="${mesh}"
-              scale="10 10 10" />
+            <mesh filename="${mesh_file}" scale="1 1 1" />
           </xacro:if>
           <xacro:unless value="${use_own_mesh}">
-            <cylinder length="0.0001" radius="0.0001"/>
+            <mesh filename="package://aeroscan_uav_simulation/meshes/propeller_${direction}.dae"
+              scale="${radius_rotor} ${radius_rotor} ${radius_rotor}" /> <!-- The propeller meshes have a radius of 1m -->
+            <!-- <box size="${2*radius_rotor} 0.01 0.005"/> -->
+            <!-- <cylinder length="0.0001" radius="0.0001"/> -->
           </xacro:unless>
         </geometry>
